Commit message: progress towards biped balance solving

File: robot/robot.urdf (robot description, URDF)
Before this commit: robot onshape, 19 links, 18 joints
Links:
- added link feet_2_sole, mass 0.01
- added link feet_sole, mass 0.01
Joints:
- added joint leg_left_sole_joint_fixed: type fixed, parent feet_2, child feet_2_sole, origin xyz=0 0 -0.015 rpy=0 0 0, axis 1 0 0
- added joint leg_right_sole_joint_fixed: type fixed, parent feet, child feet_sole, origin xyz=0 0 -0.015 rpy=0 0 0, axis 1 0 0

Commit message: added visualization within the mujoco scene to track the reference COM with the actual COM in TSID

File: robot/robot.urdf (robot description, URDF)
Before this commit: robot onshape, 21 links, 20 joints
Joints:
- joint head_pitch: limit effort=1 velocity=20 -> effort=3 velocity=4.0; origin xyz=0.013824999999999965788 0.0031093300000000073657 -0.017360000000000014309 rpy=1.570796326794896558 -1.1508559106436137405e-16 -1.570796326794896558 -> xyz=0.013824999999999965788 0.0031093300000000073657 -0.017360000000000014309 rpy=1.570796326794896558 0 -1.570796326794896558
- joint head_yaw: limit effort=1 velocity=20 -> effort=3 velocity=4.0
- joint left_ankle_pitch: limit effort=1 velocity=20 -> effort=3 velocity=4.0; origin xyz=0 -0.07621999999999998221 0 rpy=3.141592653589793116 2.4651903288156624393e-32 0 -> xyz=0 -0.07621999999999998221 0 rpy=3.141592653589793116 0 0
- joint left_elbow: limit effort=1 velocity=20 -> effort=3 velocity=4.0
- joint left_hip_pitch: limit effort=1 velocity=20 -> effort=3 velocity=4.0; origin xyz=0.040849999999999969669 0.041699969999999995929 -0.01235999999999999252 rpy=-1.570796326794896558 1.534474547524817992e-16 1.570796326794896558 -> xyz=0.040849999999999969669 0.041699969999999995929 -0.01235999999999999252 rpy=-1.570796326794896558 0 1.570796326794896558
- joint left_hip_roll: limit effort=1 velocity=20 -> effort=3 velocity=4.0
- joint left_hip_yaw: limit effort=1 velocity=20 -> effort=3 velocity=4.0; origin xyz=0 0.057449979999999997715 0.012002799999999994029 rpy=1.570796326794896558 -4.9129737742167706065e-48 0 -> xyz=0 0.057449979999999997715 0.012002799999999994029 rpy=1.570796326794896558 0 0
- joint left_knee: limit effort=1 velocity=20 -> effort=3 velocity=4.0
- joint left_shoulder_pitch: limit effort=1 velocity=20 -> effort=3 velocity=4.0
- joint left_shoulder_roll: limit effort=1 velocity=20 -> effort=3 velocity=4.0
- joint leg_left_sole_joint_fixed: origin xyz=0 0 -0.015 rpy=0 0 0 -> xyz=0 0.03 0.0275 rpy=1.57079632679 3.14159265359 0
- joint leg_right_sole_joint_fixed: origin xyz=0 0 -0.015 rpy=0 0 0 -> xyz=0 0.03 0.0275 rpy=1.57079632679 0 0
- joint right_ankle_pitch: limit effort=1 velocity=20 -> effort=3 velocity=4.0; origin xyz=0 -0.07621999999999998221 0 rpy=-3.141592653589793116 2.4651903288156618919e-32 0 -> xyz=0 -0.07621999999999998221 0 rpy=-3.141592653589793116 0 0
- joint right_elbow: limit effort=1 velocity=20 -> effort=3 velocity=4.0
- joint right_hip_pitch: limit effort=1 velocity=20 -> effort=3 velocity=4.0
- joint right_hip_roll: limit effort=1 velocity=20 -> effort=3 velocity=4.0
- joint right_hip_yaw: limit effort=1 velocity=20 -> effort=3 velocity=4.0
- joint right_knee: limit effort=1 velocity=20 -> effort=3 velocity=4.0; origin xyz=0.013049499999999991662 1.0408340855860842566e-17 -0.034359999999999987774 rpy=1.570796326794896558 -0 1.570796326794896336 -> xyz=0.013049499999999991662 1.0408340855860842566e-17 -0.034359999999999987774 rpy=1.570796326794896558 0 1.570796326794896336
- joint right_shoulder_pitch: limit effort=1 velocity=20 -> effort=3 velocity=4.0; origin xyz=-0.070850000000000037947 0.040502249999999927199 0.12166519000000000639 rpy=1.570796326794896558 -1.534474547524817992e-16 1.570796326794896558 -> xyz=-0.070850000000000037947 0.040502249999999927199 0.12166519000000000639 rpy=1.570796326794896558 0 1.570796326794896558
- joint right_shoulder_roll: limit effort=1 velocity=20 -> effort=3 velocity=4.0

Commit message: follow com reference

File: robot/robot.urdf (robot description, URDF)
Before this commit: robot onshape, 21 links, 20 joints
Joints:
- joint leg_left_sole_joint_fixed: origin xyz=0 0.03 0.0275 rpy=1.57079632679 3.14159265359 0 -> xyz=0 0.03 0.0275 rpy=1.57079632679 1.57079632679 0
- joint leg_right_sole_joint_fixed: origin xyz=0 0.03 0.0275 rpy=1.57079632679 0 0 -> xyz=0 0.03 0.0275 rpy=1.57079632679 -1.57079632679 0

Commit message: balance checkpoint

File: robot/robot.urdf (robot description, URDF)
Before this commit: robot onshape, 21 links, 20 joints
Joints:
- joint leg_left_sole_joint_fixed: origin xyz=0 0.03 0.0275 rpy=1.57079632679 1.57079632679 0 -> xyz=0 0.03 0.0275 rpy=1.57079632679 -1.57079632679 0

Commit message: fixing urdf:

File: robot/robot.urdf (robot description, URDF)
Before this commit: robot onshape, 21 links, 20 joints
Joints:
- joint leg_right_sole_joint_fixed: origin xyz=0 0.03 0.0275 rpy=1.57079632679 -1.57079632679 0 -> xyz=0 0.03 0.0275 rpy=1.57079632679 1.57079632679 0
