Commit message: clean up clean up

File: robot/v1/urdf/robot.urdf (robot description, URDF)
Before this commit: robot C:\Users\David\desktop\v1_urdf, 23 links, 22 joints
Joints:
- joint left_sole_joint_fixed: origin xyz=0 0.03 0.0275 rpy=1.57079632679 -1.57079632679 0 -> xyz=0 0.027 -0.0275 rpy=1.57079632679 1.57079632679 0
- joint right_sole_joint_fixed: origin xyz=0 0.03 0.0275 rpy=1.57079632679 1.57079632679 0 -> xyz=0 0.027 -0.0275 rpy=1.57079632679 1.57079632679 0

File: robot/v1/urdf/robot_mod.urdf (robot description, URDF)
Before this commit: robot C:\Users\David\desktop\v1_urdf, 23 links, 22 joints
Joints:
- joint left_sole_joint_fixed: origin xyz=0 0.027 -0.0275 rpy=1.57079632679 1.57079632679 0 -> xyz=0 0.027 -0.0275 rpy=1.57079632679 0 0
- joint right_sole_joint_fixed: origin xyz=0 0.027 -0.0275 rpy=1.57079632679 1.57079632679 0 -> xyz=0 0.027 -0.0275 rpy=1.57079632679 0 0
